File: MainBoard.sch (EAGLE design)
At the start: 37 parts, among them IC2 2982-DRV8825, IC3 2982-DRV8825, IC4 2982-DRV8825, IC5 2982-DRV8825

Commit message: Pin 10 on the shift registers should be pulled high to enable the outputs
Connections:
- net GND: no longer SR1A.SCL, SR2AA.SCL, SR2BA.SCL
- net VCC: now also SR1A.SCL, SR2AA.SCL, SR2BA.SCL
Changed lines of the file:
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@@
 <part name="GND24" library="supply1" library_urn="urn:adsk.eagle:library:371" deviceset="GND" device=""/>
 <part name="GND25" library="supply1" library_urn="urn:adsk.eagle:library:371" deviceset="GND" device=""/>
-<part name="GND26" library="supply1" library_urn="urn:adsk.eagle:library:371" deviceset="GND" device=""/>
 <part name="GND27" library="supply1" library_urn="urn:adsk.eagle:library:371" deviceset="GND" device=""/>
-<part name="GND28" library="supply1" library_urn="urn:adsk.eagle:library:371" deviceset="GND" device=""/>
-<part name="GND29" library="supply1" library_urn="urn:adsk.eagle:library:371" deviceset="GND" device=""/>
 <part name="P+3" library="supply1" library_urn="urn:adsk.eagle:library:371" deviceset="VCC" device=""/>
 <part name="C1" library="rcl" library_urn="urn:adsk.eagle:library:334" deviceset="C-EU" device="C0805" package3d_urn="urn:adsk.eagle:package:23617/2" value="100nF"/>
@@
 <part name="P+20" library="supply1" library_urn="urn:adsk.eagle:library:371" deviceset="VCC" device=""/>
 <part name="GND20" library="supply1" library_urn="urn:adsk.eagle:library:371" deviceset="GND" device=""/>
+<part name="P+21" library="supply1" library_urn="urn:adsk.eagle:library:371" deviceset="VCC" device=""/>
+<part name="P+22" library="supply1" library_urn="urn:adsk.eagle:library:371" deviceset="VCC" device=""/>
+<part name="P+23" library="supply1" library_urn="urn:adsk.eagle:library:371" deviceset="VCC" device=""/>
 </parts>
 <sheets>
@@
 <attribute name="VALUE" x="78.74" y="91.44" size="1.778" layer="96"/>
 </instance>
-<instance part="GND26" gate="1" x="63.5" y="109.22" smashed="yes">
-<attribute name="VALUE" x="60.96" y="106.68" size="1.778" layer="96"/>
-</instance>
 <instance part="GND27" gate="1" x="175.26" y="162.56" smashed="yes">
 <attribute name="VALUE" x="172.72" y="160.02" size="1.778" layer="96"/>
-</instance>
-<instance part="GND28" gate="1" x="160.02" y="177.8" smashed="yes">
-<attribute name="VALUE" x="157.48" y="175.26" size="1.778" layer="96"/>
-</instance>
-<instance part="GND29" gate="1" x="106.68" y="83.82" smashed="yes">
-<attribute name="VALUE" x="104.14" y="81.28" size="1.778" layer="96"/>
 </instance>
 <instance part="P+3" gate="VCC" x="187.96" y="20.32" smashed="yes">
@@
 <instance part="GND20" gate="1" x="121.92" y="185.42" smashed="yes">
 <attribute name="VALUE" x="119.38" y="182.88" size="1.778" layer="96"/>
+</instance>
+<instance part="P+21" gate="VCC" x="66.04" y="114.3" smashed="yes">
+<attribute name="VALUE" x="63.5" y="111.76" size="1.778" layer="96" rot="R90"/>
+</instance>
+<instance part="P+22" gate="VCC" x="106.68" y="88.9" smashed="yes">
+<attribute name="VALUE" x="104.14" y="86.36" size="1.778" layer="96" rot="R90"/>
+</instance>
+<instance part="P+23" gate="VCC" x="160.02" y="182.88" smashed="yes">
+<attribute name="VALUE" x="157.48" y="180.34" size="1.778" layer="96" rot="R90"/>
 </instance>
 </instances>
@@
 </segment>
 <segment>
-<pinref part="SR2A" gate="A" pin="SCL"/>
-<wire x1="81.28" y1="111.76" x2="63.5" y2="111.76" width="0.1524" layer="91"/>
-<pinref part="GND26" gate="1" pin="GND"/>
-<label x="68.58" y="111.76" size="1.778" layer="95"/>
-</segment>
-<segment>
 <pinref part="SR1" gate="A" pin="G"/>
 <pinref part="GND27" gate="1" pin="GND"/>
 <wire x1="175.26" y1="165.1" x2="177.8" y2="165.1" width="0.1524" layer="91"/>
-</segment>
-<segment>
-<pinref part="SR1" gate="A" pin="SCL"/>
-<wire x1="177.8" y1="180.34" x2="160.02" y2="180.34" width="0.1524" layer="91"/>
-<pinref part="GND28" gate="1" pin="GND"/>
-</segment>
-<segment>
-<pinref part="SR2B" gate="A" pin="SCL"/>
-<pinref part="GND29" gate="1" pin="GND"/>
-<wire x1="111.76" y1="86.36" x2="106.68" y2="86.36" width="0.1524" layer="91"/>
 </segment>
 <segment>
@@
 <pinref part="P+20" gate="VCC" pin="VCC"/>
 </segment>
-</net>
+<segment>
+<pinref part="SR2A" gate="A" pin="SCL"/>
+<wire x1="81.28" y1="111.76" x2="66.04" y2="111.76" width="0.1524" layer="91"/>
+<label x="68.58" y="111.76" size="1.778" layer="95"/>
+<pinref part="P+21" gate="VCC" pin="VCC"/>
+</segment>
+<segment>
+<pinref part="SR2B" gate="A" pin="SCL"/>
+<wire x1="111.76" y1="86.36" x2="106.68" y2="86.36" width="0.1524" layer="91"/>
+<pinref part="P+22" gate="VCC" pin="VCC"/>
+</segment>
+<segment>
+<pinref part="SR1" gate="A" pin="SCL"/>
+<wire x1="177.8" y1="180.34" x2="160.02" y2="180.34" width="0.1524" layer="91"/>
+<pinref part="P+23" gate="VCC" pin="VCC"/>
+</segment>
+</net>

Commit message: Improved the layout a little bit and add some mounting holes
Connections:
- net N$13 renamed M0-X
- net N$14 renamed M1-X
- net N$15 renamed M2-X
Changed lines of the file:
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@@
 <attribute name="VALUE" x="63.5" y="111.76" size="1.778" layer="96" rot="R90"/>
 </instance>
-<instance part="P+22" gate="VCC" x="106.68" y="88.9" smashed="yes">
-<attribute name="VALUE" x="104.14" y="86.36" size="1.778" layer="96" rot="R90"/>
+<instance part="P+22" gate="VCC" x="73.66" y="88.9" smashed="yes">
+<attribute name="VALUE" x="71.12" y="86.36" size="1.778" layer="96" rot="R90"/>
 </instance>
 <instance part="P+23" gate="VCC" x="160.02" y="182.88" smashed="yes">
@@
 <segment>
 <pinref part="SR2B" gate="A" pin="SCL"/>
-<wire x1="111.76" y1="86.36" x2="106.68" y2="86.36" width="0.1524" layer="91"/>
+<wire x1="111.76" y1="86.36" x2="73.66" y2="86.36" width="0.1524" layer="91"/>
 <pinref part="P+22" gate="VCC" pin="VCC"/>
 </segment>
@@
 </segment>
 </net>
-<net name="N$13" class="0">
+<net name="M0-X" class="0">
 <segment>
 <pinref part="JP2" gate="-3" pin="2"/>
@@
 </segment>
 </net>
-<net name="N$14" class="0">
+<net name="M1-X" class="0">
 <segment>
 <pinref part="JP2" gate="-2" pin="2"/>
@@
 </segment>
 </net>
-<net name="N$15" class="0">
+<net name="M2-X" class="0">
 <segment>
 <pinref part="JP2" gate="-1" pin="2"/>
